File: hardware/schematic/famicom-expand-usb-adapter.kicad_sch (KiCad schematic)
At the start: 16 parts, among them J1 Famicom_Expansion_DA15, J2 SFC_Port_1P, J3 SFC_Port_2P, SW1 SW_Push, U1 Arduino_Nano, U2 RaspberryPi_Pico

Commit message: Move SFC_CLOCK from D4 to A5 so all SFC signals sit on A0-A5
Keeps every new SFC controller-port wire on the analog header (A0-A5),
which is physically contiguous on the Nano and easier to route than
mixing in a separate digital pin. D4 is freed back up as a spare.

Co-Authored-By: Claude Sonnet 5 <noreply@anthropic.com>
Connections:
- net SFC_CLOCK: now also U1.24 (A5); no longer U1.7 (D4)
Changed lines of the file:
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@@
-	)
-	(wire
-		(pts (xy 157.48 167.64) (xy 152.4 167.64))
-		(stroke (width 0) (type default))
 	)
 	(wire
@@
 	(wire
 		(pts (xy 182.88 182.88) (xy 187.96 182.88))
+		(stroke (width 0) (type default))
+	)
+	(wire
+		(pts (xy 182.88 185.42) (xy 187.96 185.42))
 		(stroke (width 0) (type default))
 	)
@@
 		(effects (font (size 1.27 1.27)) (justify right))
 	)
-	(label "SFC_CLOCK"
-		(at 152.4 167.64 0)
-		(effects (font (size 1.27 1.27)) (justify right))
-	)
 	(label "OUT0"
 		(at 152.4 170.18 0)
@@
 		(effects (font (size 1.27 1.27)) (justify left))
 	)
+	(label "SFC_CLOCK"
+		(at 187.96 185.42 0)
+		(effects (font (size 1.27 1.27)) (justify left))
+	)
 	(global_label "+5V"
 		(shape input)
@@
 	)
 	(no_connect
+		(at 157.48 167.64)
+	)
+	(no_connect
 		(at 172.72 147.32)
 	)
@@
 	)
 	(no_connect
-		(at 182.88 185.42)
-	)
-	(no_connect

Commit message: Share DA15 pins 2/3 with SFC LATCH/DATA_1P (A0/A1), now physically wired
Famicom expansion pins 2/3 carry no signal on the keyboard/Zapper side, so
they're reused for the SFC controller ports' LATCH and 1P DATA lines -
same "mutually exclusive use" pattern already applied to pins 4/5. Updates
schematic, connection list, and docs to match the as-built wiring.

Co-Authored-By: Claude Sonnet 5 <noreply@anthropic.com>
Connections:
- net SFC_DATA_1P: now also J1.3
- net SFC_LATCH: now also J1.2
- no-connect marks 48 -> 46
Changed lines of the file:
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@@
+	)
+	(wire
+		(pts (xy 50.8 160.02) (xy 45.72 160.02))
+		(stroke (width 0) (type default))
+	)
+	(wire
+		(pts (xy 50.8 165.1) (xy 45.72 165.1))
+		(stroke (width 0) (type default))
 	)
 	(wire
@@
 		(shape input)
 		(at 45.72 154.94 0)
+		(effects (font (size 1.27 1.27)) (justify right))
+	)
+	(label "SFC_LATCH"
+		(at 45.72 160.02 0)
+		(effects (font (size 1.27 1.27)) (justify right))
+	)
+	(label "SFC_DATA_1P"
+		(at 45.72 165.1 0)
 		(effects (font (size 1.27 1.27)) (justify right))
 	)
@@
 	)
 	(no_connect
-		(at 50.8 160.02)
-	)
-	(no_connect
-		(at 50.8 165.1)
-	)
-	(no_connect

Commit message: Revert DA15 pin2/3 <-> A0/A1 sharing; identified as AudioOUT/IRQ
Real-hardware investigation found DA15 pins 2/3 are actually AudioOUT and
IRQ, not unused - sharing them with the SFC LATCH/DATA_1P lines would have
collided with real signals. Expansion-port side physically cut; A0-A5 are
now dedicated solely to the SFC controller ports. This also means the
Famicom keyboard/Zapper and SFC controllers can now be used at the same
time (keyboard vs Zapper still exclusive - single J1 socket).

Co-Authored-By: Claude Sonnet 5 <noreply@anthropic.com>
Connections:
- net SFC_DATA_1P: no longer J1.3
- net SFC_LATCH: no longer J1.2
- no-connect marks 46 -> 48
Changed lines of the file:
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@@
-	)
-	(wire
-		(pts (xy 50.8 160.02) (xy 45.72 160.02))
-		(stroke (width 0) (type default))
-	)
-	(wire
-		(pts (xy 50.8 165.1) (xy 45.72 165.1))
-		(stroke (width 0) (type default))
 	)
 	(wire
@@
 		(shape input)
 		(at 45.72 154.94 0)
-		(effects (font (size 1.27 1.27)) (justify right))
-	)
-	(label "SFC_LATCH"
-		(at 45.72 160.02 0)
-		(effects (font (size 1.27 1.27)) (justify right))
-	)
-	(label "SFC_DATA_1P"
-		(at 45.72 165.1 0)
 		(effects (font (size 1.27 1.27)) (justify right))
 	)
@@
 	)
 	(no_connect
+		(at 50.8 160.02)
+	)
+	(no_connect
+		(at 50.8 165.1)
+	)
+	(no_connect
